File: boards/LoconetEsp32Craddle/LoconetEsp32Craddle.kicad_pcb (KiCad board)
At the start: 4 copper layers, 95 x 71 mm, 53 parts, among them J1 SD1306 I2C/Oled, J2 RJ12, J3 RJ12, Q1 SS8050, Q2 SS8050, Q3 2N7002, Q4 2N7002, Q5 2N7002, SW1 SW_Push, SW2 SW_Push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

Commit message: Update PCB
Parts:
- J1: footprint LocoNetInterface:128x64OLED -> LocoNetInterface:ER_OLEDM0.91_1x-I2C-128x64OLED
- J2, J3: footprint LocoNetInterface:AMPHENOL_RJE0166001 -> LocoNetInterface:RJ12_AMPHENOL_RJE0166001
- U5: footprint Espressif:ESP32-DevKitC -> PCM_Espressif:ESP32-DevKitC
